Commit message: added zed 2i camera bracket to urdf

File: src/bench_robot_description/urdf/fixed_structure.urdf.xacro (robot description, xacro)
@@ -77,6 +77,33 @@
     <child link="arm_mount_link"/>
     <origin xyz="0 -0.09 ${col_h }" rpy="0 0 0"/>
-</joint>
-  <xacro:arg name="dof" default="7"/>
+  </joint>
+  <link name="camera_bracket_link">
+    <visual>
+      <origin xyz="0 0 0" rpy="0 0 0"/>
+      <geometry>
+        <mesh filename="package://bench_robot_description/meshes/zed_2i_bracket.stl" scale="0.001 0.001 0.001"/>
+      </geometry>
+      <material name="white">
+        <color rgba="1 1 1 1"/>
+      </material>
+    </visual>
+    <collision>
+      <origin xyz="0 0 0" rpy="0 0 0"/>
+      <geometry>
+        <mesh filename="package://bench_robot_description/meshes/zed_2i_bracket.stl" scale="0.001 0.001 0.001"/>
+      </geometry>
+    </collision>
+    <inertial>
+      <mass value="0.2"/>
+      <origin xyz="0 0 0"/>
+      <inertia ixx="0.0001" iyy="0.0001" izz="0.0001"
+              ixy="0" ixz="0" iyz="0"/>
+    </inertial>
+  </link>
+  <joint name="camera_bracket_joint" type="fixed">
+    <parent link="top_beam_link"/>
+    <child link="camera_bracket_link"/>
+    <origin xyz="0 0 -0.0445" rpy="1.5708 0 0"/>
+  </joint>
   <xacro:arg name="robot_ip" default="yyy.yyy.yyy.yyy"/>
   <xacro:arg name="port" default="10000"/>
@@ -91,5 +118,5 @@
       parent="arm_mount_link"
       arm="gen3"
-      dof="$(arg dof)"
+      dof="7"
       vision="false"
       prefix=""

File: src/bench_robot_description/urdf/kortex_robot.xacro (robot description, xacro)
@@ -32,5 +32,5 @@
     moveit_active:=false">
     <!-- Include and load arm macro files -->
-    <xacro:include filename="$(find bench_robot_description)/urdf/${dof}/gen3_macro.xacro" />
+    <xacro:include filename="$(find bench_robot_description)/urdf/gen3_macro.xacro" />
     <!-- Load the arm -->
     <xacro:load_arm

Commit message: create arm_controlling pkg, basic code is working

File: src/bench_robot_description/urdf/fixed_structure.urdf.xacro (robot description, xacro)
@@ -76,5 +76,5 @@
     <parent link="world"/>
     <child link="arm_mount_link"/>
-    <origin xyz="0 -0.09 ${col_h }" rpy="0 0 0"/>
+    <origin xyz="0 -0.09 ${col_h }" rpy="3.14159 0 0"/>
   </joint>
   <link name="camera_bracket_link">
@@ -138,5 +138,5 @@
       gripper_joint_name="robotiq_85_left_knuckle_joint"
       >
-      <origin xyz="0 0 0" rpy="3.14159 0 0"/>
+      <origin xyz="0 0 0" rpy="0 0 0"/>
 </xacro:load_robot>
 <xacro:if value="$(arg sim_ignition)">

Commit message: print real coordinates of end effector

File: src/bench_robot_description/urdf/fixed_structure.urdf.xacro (robot description, xacro)
@@ -72,10 +72,4 @@
     <origin xyz="${half_spacing + 0.06} 0 ${col_h}" rpy="0 0.7854 0"/>
   </joint>
-  <link name="arm_mount_link"/>
-  <joint name="chassis_to_arm_mount" type="fixed">
-    <parent link="world"/>
-    <child link="arm_mount_link"/>
-    <origin xyz="0 -0.09 ${col_h }" rpy="3.14159 0 0"/>
-  </joint>
   <link name="camera_bracket_link">
     <visual>
@@ -105,4 +99,19 @@
     <child link="camera_bracket_link"/>
     <origin xyz="0 0 -0.0445" rpy="1.5708 0 0"/>
+  </joint>
+  <xacro:include filename="$(find zed_wrapper)/urdf/zed_macro.urdf.xacro" />
+  <xacro:zed_camera name="zed2i" model="zed2i" enable_gnss="false">
+    <origin xyz="0 0 0" rpy="0 0 0"/>
+  </xacro:zed_camera>
+  <joint name="zed_2i_mount_joint" type="fixed">
+    <parent link="camera_bracket_link"/>
+    <child link="zed2i_camera_link"/>
+    <origin xyz="-0.0095 -0.0373 -0.019" rpy="0 0 -1.5708"/>
+  </joint>
+  <link name="arm_mount_link"/>
+  <joint name="chassis_to_arm_mount" type="fixed">
+    <parent link="world"/>
+    <child link="arm_mount_link"/>
+    <origin xyz="0 -0.09 ${col_h }" rpy="3.14159 0 0"/>
   </joint>
   <xacro:arg name="robot_ip" default="yyy.yyy.yyy.yyy"/>
