Commit message: added long zed bracket, change rest position

File: src/bench_robot_description/urdf/fixed_structure.urdf.xacro (robot description, xacro)
@@ -76,5 +76,5 @@
       <origin xyz="0 0 0" rpy="0 0 0"/>
       <geometry>
-        <mesh filename="package://bench_robot_description/meshes/zed_2i_bracket.stl" scale="0.001 0.001 0.001"/>
+        <mesh filename="package://bench_robot_description/meshes/zed_2i_bracket_long.stl" scale="0.001 0.001 0.001"/>
       </geometry>
       <material name="white">
@@ -85,5 +85,5 @@
       <origin xyz="0 0 0" rpy="0 0 0"/>
       <geometry>
-        <mesh filename="package://bench_robot_description/meshes/zed_2i_bracket.stl" scale="0.001 0.001 0.001"/>
+        <mesh filename="package://bench_robot_description/meshes/zed_2i_bracket_long.stl" scale="0.001 0.001 0.001"/>
       </geometry>
     </collision>
@@ -98,5 +98,5 @@
     <parent link="top_beam_link"/>
     <child link="camera_bracket_link"/>
-    <origin xyz="0 0 -0.0445" rpy="1.5708 0 0"/>
+    <origin xyz="0 0 -0.13" rpy="1.5708 0 0"/>
   </joint>
   <xacro:include filename="$(find zed_wrapper)/urdf/zed_macro.urdf.xacro" />
@@ -113,5 +113,5 @@
     <parent link="world"/>
     <child link="arm_mount_link"/>
-    <origin xyz="0 -0.09 ${col_h }" rpy="3.14159 0 0"/>
+    <origin xyz="0 -0.08 ${col_h }" rpy="3.14159 0 3.14159"/>
   </joint>
   <xacro:arg name="robot_ip" default="yyy.yyy.yyy.yyy"/>

Commit message: add the bench in urdf

File: src/bench_robot_description/urdf/fixed_structure.urdf.xacro (robot description, xacro)
@@ -5,7 +5,11 @@
   <xacro:property name="col_d" value="0.06"/>          <!-- 60 mm -->
   <xacro:property name="col_h" value="1.8288"/>        <!-- 6 ft -->
-  <xacro:property name="beam_len" value="1.524"/>      <!-- 5 ft -->
+  <xacro:property name="beam_len" value="1.0"/>        <!-- 1 m top beam -->
   <xacro:property name="beam_w" value="0.06"/>
   <xacro:property name="beam_d" value="0.06"/>
+  <xacro:property name="bench_support_len" value="1.0"/>   <!-- short support beam -->
+  <xacro:property name="bench_support_w" value="1.0"/>
+  <xacro:property name="bench_support_d" value="0.12"/>
+  <xacro:property name="bench_gap_z" value="1.0"/>        <!-- 1 m below the top beam -->
   <xacro:property name="plate_x" value="0.43"/>
   <xacro:property name="plate_y" value="0.06"/>
@@ -57,4 +61,11 @@
     <child link="top_beam_link"/>
     <origin xyz="0 0 ${col_h - beam_d/2.0}" rpy="0 0 0"/>
+  </joint>
+  <!-- ===== Bench support beam under the top beam ===== -->
+  <xacro:box_link name="bench_support_beam_link" sx="${bench_support_len}" sy="${bench_support_w}" sz="${bench_support_d}"/>
+  <joint name="base_link_to_bench_support_beam" type="fixed">
+    <parent link="world"/>
+    <child link="bench_support_beam_link"/>
+    <origin xyz="0 0 ${col_h - beam_d/2.0 - bench_gap_z}" rpy="0 0 0"/>
   </joint>
   <!-- ===== Support plates (one per column at the beam connection) ===== -->

Commit message: minor fixes

File: src/bench_robot_description/urdf/fixed_structure.urdf.xacro (robot description, xacro)
@@ -5,5 +5,5 @@
   <xacro:property name="col_d" value="0.06"/>          <!-- 60 mm -->
   <xacro:property name="col_h" value="1.8288"/>        <!-- 6 ft -->
-  <xacro:property name="beam_len" value="1.0"/>        <!-- 1 m top beam -->
+  <xacro:property name="beam_len" value="1.524"/>        <!-- 1 m top beam -->
   <xacro:property name="beam_w" value="0.06"/>
   <xacro:property name="beam_d" value="0.06"/>

Commit message: astra2 urdf added(not tested)

File: src/bench_robot_description/urdf/fixed_structure.urdf.xacro (robot description, xacro)
@@ -119,4 +119,10 @@
     <child link="zed2i_camera_link"/>
     <origin xyz="-0.0095 -0.0373 -0.019" rpy="0 0 -1.5708"/>
+  </joint>
+  <xacro:include filename="$(find orbbec_description)/urdf/astra2.urdf.xacro" />
+  <joint name="astra2_joint" type="fixed">
+      <parent link="top_beam_link"/>
+      <child link="astra2_camera_link"/>
+      <origin xyz="0 0 0" rpy="0 0 0"/>
   </joint>
   <link name="arm_mount_link"/>

Commit message: added astra 2 to urdf

File: src/bench_robot_description/urdf/fixed_structure.urdf.xacro (robot description, xacro)
@@ -120,9 +120,55 @@
     <origin xyz="-0.0095 -0.0373 -0.019" rpy="0 0 -1.5708"/>
   </joint>
-  <xacro:include filename="$(find orbbec_description)/urdf/astra2.urdf.xacro" />
   <joint name="astra2_joint" type="fixed">
       <parent link="top_beam_link"/>
       <child link="astra2_camera_link"/>
-      <origin xyz="0 0 0" rpy="0 0 0"/>
+      <origin xyz="0.03 0.06 -0.09" rpy="0 1.5708 -1.5708"/>
+  </joint>
+  <link name="astra2_camera_link">
+    <visual>
+      <origin xyz="-0.012323995999904 -0.0374999999985815 -0.0281503197112" rpy="0 0 0"/>
+      <geometry>
+        <mesh filename="package://orbbec_description/meshes/astra2/base_link.STL"/>
+      </geometry>
+      <material name="astra2_body">
+        <color rgba="0.82745 0.69804 0.4902 1"/>
+      </material>
+    </visual>
+    <collision>
+      <origin xyz="0 0 0" rpy="0 0 0"/>
+      <geometry>
+        <mesh filename="package://orbbec_description/meshes/astra2/base_link.STL"/>
+      </geometry>
+    </collision>
+    <inertial>
+      <origin xyz="-0.0160938085585399 -0.00100885505248632 0.0279919581775268" rpy="0 0 0"/>
+      <mass value="0.0101524380243699"/>
+      <inertia ixx="1.69184979927567E-05" ixy="-8.18066547859061E-09" ixz="-1.27426373196599E-09"
+               iyy="7.7096717121366E-07" iyz="1.08838945581987E-08" izz="1.61801971464778E-05"/>
+    </inertial>
+  </link>
+  <link name="astra2_depth_frame"/>
+  <joint name="astra2_depth_joint" type="fixed">
+    <parent link="astra2_camera_link"/>
+    <child link="astra2_depth_frame"/>
+    <origin xyz="0 0 0" rpy="0 0 0"/>
+  </joint>
+  <link name="astra2_depth_optical_frame"/>
+  <joint name="astra2_depth_optical_joint" type="fixed">
+    <parent link="astra2_depth_frame"/>
+    <child link="astra2_depth_optical_frame"/>
+    <origin xyz="0 0 0" rpy="-1.5707963267949 0 -1.5707963267949"/>
+  </joint>
+  <link name="astra2_color_frame"/>
+  <joint name="astra2_color_joint" type="fixed">
+    <parent link="astra2_depth_frame"/>
+    <child link="astra2_color_frame"/>
+    <origin xyz="0.0025420000310987234 -0.01850000023841858 0" rpy="0 0 0"/>
+  </joint>
+  <link name="astra2_color_optical_frame"/>
+  <joint name="astra2_color_optical_joint" type="fixed">
+    <parent link="astra2_color_frame"/>
+    <child link="astra2_color_optical_frame"/>
+    <origin xyz="0 0 0" rpy="-1.5707963267949 0 -1.5707963267949"/>
   </joint>
   <link name="arm_mount_link"/>

Commit message: added gemini 335, remove astra

File: src/bench_robot_description/urdf/fixed_structure.urdf.xacro (robot description, xacro)
@@ -120,17 +120,17 @@
     <origin xyz="-0.0095 -0.0373 -0.019" rpy="0 0 -1.5708"/>
   </joint>
-  <joint name="astra2_joint" type="fixed">
+  <joint name="gemini335_joint" type="fixed">
       <parent link="top_beam_link"/>
-      <child link="astra2_camera_link"/>
+      <child link="gemini335_camera_link"/>
       <origin xyz="0.03 0.06 -0.09" rpy="0 1.5708 -1.5708"/>
   </joint>
-  <link name="astra2_camera_link">
+  <link name="gemini335_camera_link">
     <visual>
-      <origin xyz="-0.012323995999904 -0.0374999999985815 -0.0281503197112" rpy="0 0 0"/>
-      <geometry>
-        <mesh filename="package://orbbec_description/meshes/astra2/base_link.STL"/>
-      </geometry>
-      <material name="astra2_body">
-        <color rgba="0.82745 0.69804 0.4902 1"/>
+      <origin xyz="-0.01587 -0.025 -0.0125" rpy="0 0 0"/>
+      <geometry>
+        <mesh filename="package://orbbec_description/meshes/gemini335_336/camera_link.STL"/>
+      </geometry>
+      <material name="gemini335_body">
+        <color rgba="1 1 1 1"/>
       </material>
     </visual>
@@ -138,36 +138,36 @@
       <origin xyz="0 0 0" rpy="0 0 0"/>
       <geometry>
-        <mesh filename="package://orbbec_description/meshes/astra2/base_link.STL"/>
+        <mesh filename="package://orbbec_description/meshes/gemini335_336/camera_link.STL"/>
       </geometry>
     </collision>
     <inertial>
-      <origin xyz="-0.0160938085585399 -0.00100885505248632 0.0279919581775268" rpy="0 0 0"/>
-      <mass value="0.0101524380243699"/>
-      <inertia ixx="1.69184979927567E-05" ixy="-8.18066547859061E-09" ixz="-1.27426373196599E-09"
-               iyy="7.7096717121366E-07" iyz="1.08838945581987E-08" izz="1.61801971464778E-05"/>
+      <origin xyz="0.00277269933215555 -0.0000106084680351007 0.012801025085723" rpy="0 0 0"/>
+      <mass value="0.0186143499064346"/>
+      <inertia ixx="1.38922229644605E-05" ixy="-4.74617876641156E-09" ixz="1.99175628166615E-08"
+               iyy="1.70686808598814E-06" iyz="-7.18717290327325E-09" izz="1.31766831843134E-05"/>
     </inertial>
   </link>
-  <link name="astra2_depth_frame"/>
-  <joint name="astra2_depth_joint" type="fixed">
-    <parent link="astra2_camera_link"/>
-    <child link="astra2_depth_frame"/>
+  <link name="gemini335_depth_frame"/>
+  <joint name="gemini335_depth_joint" type="fixed">
+    <parent link="gemini335_camera_link"/>
+    <child link="gemini335_depth_frame"/>
     <origin xyz="0 0 0" rpy="0 0 0"/>
   </joint>
-  <link name="astra2_depth_optical_frame"/>
-  <joint name="astra2_depth_optical_joint" type="fixed">
-    <parent link="astra2_depth_frame"/>
-    <child link="astra2_depth_optical_frame"/>
+  <link name="gemini335_depth_optical_frame"/>
+  <joint name="gemini335_depth_optical_joint" type="fixed">
+    <parent link="gemini335_depth_frame"/>
+    <child link="gemini335_depth_optical_frame"/>
     <origin xyz="0 0 0" rpy="-1.5707963267949 0 -1.5707963267949"/>
   </joint>
-  <link name="astra2_color_frame"/>
-  <joint name="astra2_color_joint" type="fixed">
-    <parent link="astra2_depth_frame"/>
-    <child link="astra2_color_frame"/>
-    <origin xyz="0.0025420000310987234 -0.01850000023841858 0" rpy="0 0 0"/>
-  </joint>
-  <link name="astra2_color_optical_frame"/>
-  <joint name="astra2_color_optical_joint" type="fixed">
-    <parent link="astra2_color_frame"/>
-    <child link="astra2_color_optical_frame"/>
+  <link name="gemini335_color_frame"/>
+  <joint name="gemini335_color_joint" type="fixed">
+    <parent link="gemini335_depth_frame"/>
+    <child link="gemini335_color_frame"/>
+    <origin xyz="0.001663 -0.014005 0.000005" rpy="0 0 0"/>
+  </joint>
+  <link name="gemini335_color_optical_frame"/>
+  <joint name="gemini335_color_optical_joint" type="fixed">
+    <parent link="gemini335_color_frame"/>
+    <child link="gemini335_color_optical_frame"/>
     <origin xyz="0 0 0" rpy="-1.5707963267949 0 -1.5707963267949"/>
   </joint>

Commit message: minor fixes

File: src/bench_robot_description/urdf/fixed_structure.urdf.xacro (robot description, xacro)
@@ -123,5 +123,5 @@
       <parent link="top_beam_link"/>
       <child link="gemini335_camera_link"/>
-      <origin xyz="0.03 0.06 -0.09" rpy="0 1.5708 -1.5708"/>
+      <origin xyz="-0.03 0.055 -0.09" rpy="0 1.5708 1.5708"/>
   </joint>
   <link name="gemini335_camera_link">

Commit message: joint limits applied

File: src/bench_robot_description/urdf/fixed_structure.urdf.xacro (robot description, xacro)
@@ -10,6 +10,6 @@
   <xacro:property name="bench_support_len" value="1.0"/>   <!-- short support beam -->
   <xacro:property name="bench_support_w" value="1.0"/>
-  <xacro:property name="bench_support_d" value="0.12"/>
-  <xacro:property name="bench_gap_z" value="1.0"/>        <!-- 1 m below the top beam -->
+  <xacro:property name="bench_support_d" value="0.01"/>
+  <xacro:property name="bench_gap_z" value="0.95"/>        <!-- 1 m below the top beam -->
   <xacro:property name="plate_x" value="0.43"/>
   <xacro:property name="plate_y" value="0.06"/>

File: src/bench_robot_description/urdf/gen3_macro.xacro (robot description, xacro)
@@ -28,5 +28,5 @@
     isaac_joint_commands:=/isaac_joint_commands
     isaac_joint_states:=/isaac_joint_states
-    use_external_cable:=false
+    use_external_cable:=true
     initial_positions:=${dict(joint_1=0.0,joint_2=0.0,joint_3=0.0,joint_4=0.0,joint_5=0.0,joint_6=0.0,joint_7=0.0)}
     moveit_active:=false">
@@ -117,6 +117,6 @@
           xyz="0 0 1" />
         <limit
-          lower="${-2*PI}"
-          upper="${2*PI}"
+          lower="${-PI}"
+          upper="${PI}"
           effort="39"
           velocity="1.3963" />
@@ -207,6 +207,6 @@
           xyz="0 0 1" />
         <limit
-          lower="${-2*PI}"
-          upper="${2*PI}"
+          lower="${-PI}"
+          upper="${PI}"
           effort="39"
           velocity="1.3963" />
@@ -297,6 +297,6 @@
           xyz="0 0 1" />
         <limit
-          lower="${-2*PI}"
-          upper="${2*PI}"
+          lower="${-PI}"
+          upper="${PI}"
           effort="9"
           velocity="1.2218" />
@@ -413,6 +413,6 @@
           xyz="0 0 1" />
         <limit
-          lower="${-2*PI}"
-          upper="${2*PI}"
+          lower="${-PI}"
+          upper="${PI}"
           effort="9"
           velocity="1.2218" />

File: src/bench_robot_description/urdf/kortex_robot.xacro (robot description, xacro)
@@ -25,5 +25,5 @@
     isaac_joint_commands:=/isaac_joint_commands
     isaac_joint_states:=/isaac_joint_states
-    use_external_cable:=false
+    use_external_cable:=true
     initial_positions:=${dict(joint_1=0.0,joint_2=-1.877,joint_3=0.0,joint_4=0.792,joint_5=0.0,joint_6=1.096,joint_7=0.0)}
     gripper_max_velocity:=100.0

Commit message: added new obbec 336 camera to urdf

File: src/bench_robot_description/urdf/fixed_structure.urdf.xacro (robot description, xacro)
@@ -83,4 +83,5 @@
     <origin xyz="${half_spacing + 0.06} 0 ${col_h}" rpy="0 0.7854 0"/>
   </joint>
+  <!-- Top-beam ZED 2i bracket and camera mount disabled.
   <link name="camera_bracket_link">
     <visual>
@@ -120,4 +121,5 @@
     <origin xyz="-0.0095 -0.0373 -0.019" rpy="0 0 -1.5708"/>
   </joint>
+  -->
   <joint name="gemini335_joint" type="fixed">
       <parent link="top_beam_link"/>

File: src/bench_robot_description/urdf/gen3_macro.xacro (robot description, xacro)
@@ -456,9 +456,41 @@
       <origin xyz="0.0133 0 0.012" rpy="0 -1.5708 0"/>
     </joint>-->
-    <xacro:include filename="$(find orbbec_description)/urdf/gemini_335_336.urdf.xacro" />
-    <joint name="orbbec_mount_joint" type="fixed">
+    <!-- Local copy fixes the upstream camera_link visual/collision mismatch. -->
+    <xacro:include filename="$(find bench_robot_description)/urdf/gemini_335_336_aligned.urdf.xacro" />
+    <!--
+      The centered bracket STL is in millimetres and has its bounding-box
+      center at the bracket link origin. This makes joint rotations occur
+      about the center of the bracket instead of the Fusion assembly origin.
+    -->
+    <link name="${prefix}ee_camera_bracket_link">
+      <visual>
+        <origin xyz="0 0 0" rpy="0 0 0"/>
+        <geometry>
+          <mesh
+            filename="package://bench_robot_description/meshes/EE_camera_bracket_centered.stl"
+            scale="0.001 0.001 0.001"/>
+        </geometry>
+        <material name="ee_camera_bracket_material">
+          <color rgba="0.15 0.15 0.15 1.0"/>
+        </material>
+      </visual>
+      <collision>
+        <origin xyz="0 0 0" rpy="0 0 0"/>
+        <geometry>
+          <mesh
+            filename="package://bench_robot_description/meshes/EE_camera_bracket_centered.stl"
+            scale="0.001 0.001 0.001"/>
+        </geometry>
+      </collision>
+    </link>
+    <joint name="${prefix}ee_camera_bracket_joint" type="fixed">
       <parent link="${prefix}end_effector_link"/>
+      <child link="${prefix}ee_camera_bracket_link"/>
+      <origin xyz="0 -0.009 -0.012" rpy="0 0 3.1416"/>
+    </joint>
+    <joint name="${prefix}orbbec_mount_joint" type="fixed">
+      <parent link="${prefix}ee_camera_bracket_link"/>
       <child link="camera_link"/>
-      <origin xyz="0 0.025 0.03" rpy="0 -1.5708 0"/>
+      <origin xyz="0.025 0.045 0.015" rpy="-1.5708 -1.5708 0"/>
     </joint>
   </xacro:macro>
