Commit message: fix orbbec camera joint

File: src/bench_robot_description/urdf/gen3_macro.xacro (robot description, xacro)
@@ -460,5 +460,5 @@
       <parent link="${prefix}end_effector_link"/>
       <child link="camera_link"/>
-      <origin xyz="0 0 0.02" rpy="0 -1.5708 0"/>
+      <origin xyz="0 0.025 0.03" rpy="0 -1.5708 0"/>
     </joint>
   </xacro:macro>
