Commit message: minor fixes

File: src/bench_robot_description/urdf/gemini_335_336_aligned.urdf.xacro (robot description, xacro)
@@ -6,5 +6,5 @@
 <robot xmlns:xacro="http://ros.org/wiki/xacro" name="gemini_335_336">
     <xacro:property name="mesh_path" value="package://orbbec_description/meshes/gemini335_336/" />
-    <link name="camera_link">
+    <link name="gemini336_link">
         <inertial>
             <origin xyz="0.00277269933215555 -1.06084680351007E-05 0.012801025085723" rpy="0 0 0" />
@@ -31,5 +31,5 @@
         </collision>
     </link>
-    <link name="camera_bottom_screw_frame">
+    <link name="gemini336_bottom_screw_frame">
         <inertial>
             <origin xyz="0.00255168206289301 -0.00123934714960528 0.0118889875786098" rpy="0 0 0" />
@@ -42,5 +42,5 @@
             <origin xyz="0 0 0" rpy="0 0 0" />
             <geometry>
-                <mesh filename="${mesh_path}camera_bottom_screw_frame.STL" />
+                <mesh filename="${mesh_path}gemini336_bottom_screw_frame.STL" />
             </geometry>
             <material name="">
@@ -51,5 +51,5 @@
             <origin xyz="0 0 0" rpy="0 0 0" />
             <geometry>
-                <mesh filename="${mesh_path}camera_bottom_screw_frame.STL" />
+                <mesh filename="${mesh_path}gemini336_bottom_screw_frame.STL" />
             </geometry>
         </collision>
@@ -57,9 +57,9 @@
     <joint name="camera_bottom_screw_frame_joint" type="fixed">
         <origin xyz="-0.01587 -0.025 -0.0125" rpy="0 0 0" />
-        <parent link="camera_link" />
-        <child link="camera_bottom_screw_frame" />
-        <axis xyz="0 0 0" />
-    </joint>
-    <link name="camera_left_ir_frame">
+        <parent link="gemini336_link" />
+        <child link="gemini336_bottom_screw_frame" />
+        <axis xyz="0 0 0" />
+    </joint>
+    <link name="gemini336_left_ir_frame">
         <inertial>
             <origin xyz="-0.00158020887627678 -1.52683853303637E-08 -1.4860800305164E-07"
@@ -73,14 +73,14 @@
             <origin xyz="-25 0 0" rpy="0 0 0" />
             <geometry>
-                <mesh filename="${mesh_path}camera_left_ir_frame.STL" />
-            </geometry>
-            <material name="">
-                <color rgba="0.501960784313725 0.250980392156863 0.250980392156863 1" />
-            </material>
-        </visual>
-        <collision>
-            <origin xyz="0 0 0" rpy="0 0 0" />
-            <geometry>
-                <mesh filename="${mesh_path}camera_left_ir_frame.STL" />
+                <mesh filename="${mesh_path}gemini336_left_ir_frame.STL" />
+            </geometry>
+            <material name="">
+                <color rgba="0.501960784313725 0.250980392156863 0.250980392156863 1" />
+            </material>
+        </visual>
+        <collision>
+            <origin xyz="0 0 0" rpy="0 0 0" />
+            <geometry>
+                <mesh filename="${mesh_path}gemini336_left_ir_frame.STL" />
             </geometry>
         </collision>
@@ -88,9 +88,9 @@
     <joint name="camera_left_ir_joint" type="fixed">
         <origin xyz="0 0 0" rpy="0 0 0" />
-        <parent link="camera_depth_frame" />
-        <child link="camera_left_ir_frame" />
-        <axis xyz="0 0 0" />
-    </joint>
-    <link name="camera_left_ir_optical_frame">
+        <parent link="gemini336_depth_frame" />
+        <child link="gemini336_left_ir_frame" />
+        <axis xyz="0 0 0" />
+    </joint>
+    <link name="gemini336_left_ir_optical_frame">
         <inertial>
             <origin xyz="1.52683853338331E-08 1.48608003051636E-07 -0.00158020887627678" rpy="0 0 0" />
@@ -103,14 +103,14 @@
             <origin xyz="0 0 0" rpy="0 0 0" />
             <geometry>
-                <mesh filename="${mesh_path}camera_left_ir_optical_frame.STL" />
-            </geometry>
-            <material name="">
-                <color rgba="0.501960784313725 0.250980392156863 0.250980392156863 1" />
-            </material>
-        </visual>
-        <collision>
-            <origin xyz="0 0 0" rpy="0 0 0" />
-            <geometry>
-                <mesh filename="${mesh_path}camera_left_ir_optical_frame.STL" />
+                <mesh filename="${mesh_path}gemini336_left_ir_optical_frame.STL" />
+            </geometry>
+            <material name="">
+                <color rgba="0.501960784313725 0.250980392156863 0.250980392156863 1" />
+            </material>
+        </visual>
+        <collision>
+            <origin xyz="0 0 0" rpy="0 0 0" />
+            <geometry>
+                <mesh filename="${mesh_path}gemini336_left_ir_optical_frame.STL" />
             </geometry>
         </collision>
@@ -118,9 +118,9 @@
     <joint name="camera_left_ir_optical_joint" type="fixed">
         <origin xyz="0 0 0" rpy="-1.5707963267949 0 -1.5707963267949" />
-        <parent link="camera_left_ir_frame" />
-        <child link="camera_left_ir_optical_frame" />
-        <axis xyz="0 0 0" />
-    </joint>
-    <link name="camera_right_ir_frame">
+        <parent link="gemini336_left_ir_frame" />
+        <child link="gemini336_left_ir_optical_frame" />
+        <axis xyz="0 0 0" />
+    </joint>
+    <link name="gemini336_right_ir_frame">
         <inertial>
             <origin xyz="-0.00158020887627678 -1.52683853303637E-08 -1.48608003050581E-07"
@@ -134,14 +134,14 @@
             <origin xyz="0 0 0" rpy="0 0 0" />
             <geometry>
-                <mesh filename="${mesh_path}camera_right_ir_frame.STL" />
-            </geometry>
-            <material name="">
-                <color rgba="0.501960784313725 0.250980392156863 0.250980392156863 1" />
-            </material>
-        </visual>
-        <collision>
-            <origin xyz="0 0 0" rpy="0 0 0" />
-            <geometry>
-                <mesh filename="${mesh_path}camera_right_ir_frame.STL" />
+                <mesh filename="${mesh_path}gemini336_right_ir_frame.STL" />
+            </geometry>
+            <material name="">
+                <color rgba="0.501960784313725 0.250980392156863 0.250980392156863 1" />
+            </material>
+        </visual>
+        <collision>
+            <origin xyz="0 0 0" rpy="0 0 0" />
+            <geometry>
+                <mesh filename="${mesh_path}gemini336_right_ir_frame.STL" />
             </geometry>
         </collision>
@@ -149,9 +149,9 @@
     <joint name="camera_right_ir_joint" type="fixed">
         <origin xyz="0 -0.05 0" rpy="0 0 0" />
-        <parent link="camera_depth_frame" />
-        <child link="camera_right_ir_frame" />
-        <axis xyz="0 0 0" />
-    </joint>
-    <link name="camera_right_ir_optical_frame">
+        <parent link="gemini336_depth_frame" />
+        <child link="gemini336_right_ir_frame" />
+        <axis xyz="0 0 0" />
+    </joint>
+    <link name="gemini336_right_ir_optical_frame">
         <inertial>
             <origin xyz="1.52683853268942E-08 1.4860800305058E-07 -0.00158020887627678" rpy="0 0 0" />
@@ -164,14 +164,14 @@
             <origin xyz="0 0 0" rpy="0 0 0" />
             <geometry>
-                <mesh filename="${mesh_path}camera_right_ir_optical_frame.STL" />
-            </geometry>
-            <material name="">
-                <color rgba="0.501960784313725 0.250980392156863 0.250980392156863 1" />
-            </material>
-        </visual>
-        <collision>
-            <origin xyz="0 0 0" rpy="0 0 0" />
-            <geometry>
-                <mesh filename="${mesh_path}camera_right_ir_optical_frame.STL" />
+                <mesh filename="${mesh_path}gemini336_right_ir_optical_frame.STL" />
+            </geometry>
+            <material name="">
+                <color rgba="0.501960784313725 0.250980392156863 0.250980392156863 1" />
+            </material>
+        </visual>
+        <collision>
+            <origin xyz="0 0 0" rpy="0 0 0" />
+            <geometry>
+                <mesh filename="${mesh_path}gemini336_right_ir_optical_frame.STL" />
             </geometry>
         </collision>
@@ -179,9 +179,9 @@
     <joint name="camera_right_ir_optical_joint" type="fixed">
         <origin xyz="0 0 0" rpy="-1.5707963267949 0 -1.5707963267949" />
-        <parent link="camera_right_ir_frame" />
-        <child link="camera_right_ir_optical_frame" />
-        <axis xyz="0 0 0" />
-    </joint>
-    <link name="camera_color_frame">
+        <parent link="gemini336_right_ir_frame" />
+        <child link="gemini336_right_ir_optical_frame" />
+        <axis xyz="0 0 0" />
+    </joint>
+    <link name="gemini336_color_frame">
         <inertial>
             <origin xyz="-0.00177079701156752 -2.20101367029782E-07 2.09893364599916E-07"
@@ -195,14 +195,14 @@
             <origin xyz="0 0 0" rpy="0 0 0" />
             <geometry>
-                <mesh filename="${mesh_path}camera_color_frame.STL" />
-            </geometry>
-            <material name="">
-                <color rgba="0.501960784313725 0.250980392156863 0.250980392156863 1" />
-            </material>
-        </visual>
-        <collision>
-            <origin xyz="0 0 0" rpy="0 0 0" />
-            <geometry>
-                <mesh filename="${mesh_path}camera_color_frame.STL" />
+                <mesh filename="${mesh_path}gemini336_color_frame.STL" />
+            </geometry>
+            <material name="">
+                <color rgba="0.501960784313725 0.250980392156863 0.250980392156863 1" />
+            </material>
+        </visual>
+        <collision>
+            <origin xyz="0 0 0" rpy="0 0 0" />
+            <geometry>
+                <mesh filename="${mesh_path}gemini336_color_frame.STL" />
             </geometry>
         </collision>
@@ -210,9 +210,9 @@
     <joint name="camera_color_joint" type="fixed">
         <origin xyz="0.001663 -0.014005 0.000005" rpy="0 0 0" />
-        <parent link="camera_depth_frame" />
-        <child link="camera_color_frame" />
-        <axis xyz="0 0 0" />
-    </joint>
-    <link name="camera_color_optical_frame">
+        <parent link="gemini336_depth_frame" />
+        <child link="gemini336_color_frame" />
+        <axis xyz="0 0 0" />
+    </joint>
+    <link name="gemini336_color_optical_frame">
         <inertial>
             <origin xyz="2.20101367029782E-07 -2.09893364599916E-07 -0.00177079701156752"
@@ -226,14 +226,14 @@
             <origin xyz="0 0 0" rpy="0 0 0" />
             <geometry>
-                <mesh filename="${mesh_path}camera_color_optical_frame.STL" />
-            </geometry>
-            <material name="">
-                <color rgba="0.501960784313725 0.250980392156863 0.250980392156863 1" />
-            </material>
-        </visual>
-        <collision>
-            <origin xyz="0 0 0" rpy="0 0 0" />
-            <geometry>
-                <mesh filename="${mesh_path}camera_color_optical_frame.STL" />
+                <mesh filename="${mesh_path}gemini336_color_optical_frame.STL" />
+            </geometry>
+            <material name="">
+                <color rgba="0.501960784313725 0.250980392156863 0.250980392156863 1" />
+            </material>
+        </visual>
+        <collision>
+            <origin xyz="0 0 0" rpy="0 0 0" />
+            <geometry>
+                <mesh filename="${mesh_path}gemini336_color_optical_frame.STL" />
             </geometry>
         </collision>
@@ -241,9 +241,9 @@
     <joint name="camera_color_optical_joint" type="fixed">
         <origin xyz="0 0 0" rpy="-1.5707963267949 0 -1.5707963267949" />
-        <parent link="camera_color_frame" />
-        <child link="camera_color_optical_frame" />
-        <axis xyz="0 0 0" />
-    </joint>
-    <link name="camera_depth_frame">
+        <parent link="gemini336_color_frame" />
+        <child link="gemini336_color_optical_frame" />
+        <axis xyz="0 0 0" />
+    </joint>
+    <link name="gemini336_depth_frame">
         <inertial>
             <origin xyz="-0.00158020887627678 -1.52683853338331E-08 -1.48608003051662E-07"
@@ -257,14 +257,14 @@
             <origin xyz="0 0 0" rpy="0 0 0" />
             <geometry>
-                <mesh filename="${mesh_path}camera_depth_frame.STL" />
-            </geometry>
-            <material name="">
-                <color rgba="0.501960784313725 0.250980392156863 0.250980392156863 1" />
-            </material>
-        </visual>
-        <collision>
-            <origin xyz="0 0 0" rpy="0 0 0" />
-            <geometry>
-                <mesh filename="${mesh_path}camera_depth_frame.STL" />
+                <mesh filename="${mesh_path}gemini336_depth_frame.STL" />
+            </geometry>
+            <material name="">
+                <color rgba="0.501960784313725 0.250980392156863 0.250980392156863 1" />
+            </material>
+        </visual>
+        <collision>
+            <origin xyz="0 0 0" rpy="0 0 0" />
+            <geometry>
+                <mesh filename="${mesh_path}gemini336_depth_frame.STL" />
             </geometry>
         </collision>
@@ -272,9 +272,9 @@
     <joint name="camera_depth_joint" type="fixed">
         <origin xyz="0 0 0" rpy="0 0 0" />
-        <parent link="camera_link" />
-        <child link="camera_depth_frame" />
-        <axis xyz="0 0 0" />
-    </joint>
-    <link name="camera_depth_optical_frame">
+        <parent link="gemini336_link" />
+        <child link="gemini336_depth_frame" />
+        <axis xyz="0 0 0" />
+    </joint>
+    <link name="gemini336_depth_optical_frame">
         <inertial>
             <origin xyz="1.52683853338331E-08 1.4860800305165E-07 -0.00158020887627678" rpy="0 0 0" />
@@ -286,14 +286,14 @@
             <origin xyz="0 0 0" rpy="0 0 0" />
             <geometry>
-                <mesh filename="${mesh_path}camera_depth_optical_frame.STL" />
-            </geometry>
-            <material name="">
-                <color rgba="0.501960784313725 0.250980392156863 0.250980392156863 1" />
-            </material>
-        </visual>
-        <collision>
-            <origin xyz="0 0 0" rpy="0 0 0" />
-            <geometry>
-                <mesh filename="${mesh_path}camera_depth_optical_frame.STL" />
+                <mesh filename="${mesh_path}gemini336_depth_optical_frame.STL" />
+            </geometry>
+            <material name="">
+                <color rgba="0.501960784313725 0.250980392156863 0.250980392156863 1" />
+            </material>
+        </visual>
+        <collision>
+            <origin xyz="0 0 0" rpy="0 0 0" />
+            <geometry>
+                <mesh filename="${mesh_path}gemini336_depth_optical_frame.STL" />
             </geometry>
         </collision>
@@ -301,6 +301,6 @@
     <joint name="camera_depth_optical_joint" type="fixed">
         <origin xyz="0 0 0" rpy="-1.5707963267949 0 -1.5707963267949" />
-        <parent link="camera_depth_frame" />
-        <child link="camera_depth_optical_frame" />
+        <parent link="gemini336_depth_frame" />
+        <child link="gemini336_depth_optical_frame" />
         <axis xyz="0 0 0" />
     </joint>

File: src/bench_robot_description/urdf/gen3_macro.xacro (robot description, xacro)
@@ -456,5 +456,5 @@
       <origin xyz="0.0133 0 0.012" rpy="0 -1.5708 0"/>
     </joint>-->
-    <!-- Local copy fixes the upstream camera_link visual/collision mismatch. -->
+    <!-- Local copy fixes the upstream gemini336_link visual/collision mismatch. -->
     <xacro:include filename="$(find bench_robot_description)/urdf/gemini_335_336_aligned.urdf.xacro" />
     <!--
@@ -491,5 +491,5 @@
     <joint name="${prefix}orbbec_mount_joint" type="fixed">
       <parent link="${prefix}ee_camera_bracket_link"/>
-      <child link="camera_link"/>
+      <child link="gemini336_link"/>
       <origin xyz="0.025 0.045 0.015" rpy="-1.5708 -1.5708 0"/>
     </joint>
