Commit message: minor adjustment

File: src/bench_robot_description/urdf/gemini_335_336_aligned.urdf.xacro (robot description, xacro)
@@ -42,5 +42,5 @@
             <origin xyz="0 0 0" rpy="0 0 0" />
             <geometry>
-                <mesh filename="${mesh_path}gemini336_bottom_screw_frame.STL" />
+                <mesh filename="${mesh_path}camera_bottom_screw_frame.STL" />
             </geometry>
             <material name="">
@@ -51,5 +51,5 @@
             <origin xyz="0 0 0" rpy="0 0 0" />
             <geometry>
-                <mesh filename="${mesh_path}gemini336_bottom_screw_frame.STL" />
+                <mesh filename="${mesh_path}camera_bottom_screw_frame.STL" />
             </geometry>
         </collision>
@@ -73,14 +73,14 @@
             <origin xyz="-25 0 0" rpy="0 0 0" />
             <geometry>
-                <mesh filename="${mesh_path}gemini336_left_ir_frame.STL" />
-            </geometry>
-            <material name="">
-                <color rgba="0.501960784313725 0.250980392156863 0.250980392156863 1" />
-            </material>
-        </visual>
-        <collision>
-            <origin xyz="0 0 0" rpy="0 0 0" />
-            <geometry>
-                <mesh filename="${mesh_path}gemini336_left_ir_frame.STL" />
+                <mesh filename="${mesh_path}camera_left_ir_frame.STL" />
+            </geometry>
+            <material name="">
+                <color rgba="0.501960784313725 0.250980392156863 0.250980392156863 1" />
+            </material>
+        </visual>
+        <collision>
+            <origin xyz="0 0 0" rpy="0 0 0" />
+            <geometry>
+                <mesh filename="${mesh_path}camera_left_ir_frame.STL" />
             </geometry>
         </collision>
@@ -103,14 +103,14 @@
             <origin xyz="0 0 0" rpy="0 0 0" />
             <geometry>
-                <mesh filename="${mesh_path}gemini336_left_ir_optical_frame.STL" />
-            </geometry>
-            <material name="">
-                <color rgba="0.501960784313725 0.250980392156863 0.250980392156863 1" />
-            </material>
-        </visual>
-        <collision>
-            <origin xyz="0 0 0" rpy="0 0 0" />
-            <geometry>
-                <mesh filename="${mesh_path}gemini336_left_ir_optical_frame.STL" />
+                <mesh filename="${mesh_path}camera_left_ir_optical_frame.STL" />
+            </geometry>
+            <material name="">
+                <color rgba="0.501960784313725 0.250980392156863 0.250980392156863 1" />
+            </material>
+        </visual>
+        <collision>
+            <origin xyz="0 0 0" rpy="0 0 0" />
+            <geometry>
+                <mesh filename="${mesh_path}camera_left_ir_optical_frame.STL" />
             </geometry>
         </collision>
@@ -134,14 +134,14 @@
             <origin xyz="0 0 0" rpy="0 0 0" />
             <geometry>
-                <mesh filename="${mesh_path}gemini336_right_ir_frame.STL" />
-            </geometry>
-            <material name="">
-                <color rgba="0.501960784313725 0.250980392156863 0.250980392156863 1" />
-            </material>
-        </visual>
-        <collision>
-            <origin xyz="0 0 0" rpy="0 0 0" />
-            <geometry>
-                <mesh filename="${mesh_path}gemini336_right_ir_frame.STL" />
+                <mesh filename="${mesh_path}camera_right_ir_frame.STL" />
+            </geometry>
+            <material name="">
+                <color rgba="0.501960784313725 0.250980392156863 0.250980392156863 1" />
+            </material>
+        </visual>
+        <collision>
+            <origin xyz="0 0 0" rpy="0 0 0" />
+            <geometry>
+                <mesh filename="${mesh_path}camera_right_ir_frame.STL" />
             </geometry>
         </collision>
@@ -164,14 +164,14 @@
             <origin xyz="0 0 0" rpy="0 0 0" />
             <geometry>
-                <mesh filename="${mesh_path}gemini336_right_ir_optical_frame.STL" />
-            </geometry>
-            <material name="">
-                <color rgba="0.501960784313725 0.250980392156863 0.250980392156863 1" />
-            </material>
-        </visual>
-        <collision>
-            <origin xyz="0 0 0" rpy="0 0 0" />
-            <geometry>
-                <mesh filename="${mesh_path}gemini336_right_ir_optical_frame.STL" />
+                <mesh filename="${mesh_path}camera_right_ir_optical_frame.STL" />
+            </geometry>
+            <material name="">
+                <color rgba="0.501960784313725 0.250980392156863 0.250980392156863 1" />
+            </material>
+        </visual>
+        <collision>
+            <origin xyz="0 0 0" rpy="0 0 0" />
+            <geometry>
+                <mesh filename="${mesh_path}camera_right_ir_optical_frame.STL" />
             </geometry>
         </collision>
@@ -195,14 +195,14 @@
             <origin xyz="0 0 0" rpy="0 0 0" />
             <geometry>
-                <mesh filename="${mesh_path}gemini336_color_frame.STL" />
-            </geometry>
-            <material name="">
-                <color rgba="0.501960784313725 0.250980392156863 0.250980392156863 1" />
-            </material>
-        </visual>
-        <collision>
-            <origin xyz="0 0 0" rpy="0 0 0" />
-            <geometry>
-                <mesh filename="${mesh_path}gemini336_color_frame.STL" />
+                <mesh filename="${mesh_path}camera_color_frame.STL" />
+            </geometry>
+            <material name="">
+                <color rgba="0.501960784313725 0.250980392156863 0.250980392156863 1" />
+            </material>
+        </visual>
+        <collision>
+            <origin xyz="0 0 0" rpy="0 0 0" />
+            <geometry>
+                <mesh filename="${mesh_path}camera_color_frame.STL" />
             </geometry>
         </collision>
@@ -226,14 +226,14 @@
             <origin xyz="0 0 0" rpy="0 0 0" />
             <geometry>
-                <mesh filename="${mesh_path}gemini336_color_optical_frame.STL" />
-            </geometry>
-            <material name="">
-                <color rgba="0.501960784313725 0.250980392156863 0.250980392156863 1" />
-            </material>
-        </visual>
-        <collision>
-            <origin xyz="0 0 0" rpy="0 0 0" />
-            <geometry>
-                <mesh filename="${mesh_path}gemini336_color_optical_frame.STL" />
+                <mesh filename="${mesh_path}camera_color_optical_frame.STL" />
+            </geometry>
+            <material name="">
+                <color rgba="0.501960784313725 0.250980392156863 0.250980392156863 1" />
+            </material>
+        </visual>
+        <collision>
+            <origin xyz="0 0 0" rpy="0 0 0" />
+            <geometry>
+                <mesh filename="${mesh_path}camera_color_optical_frame.STL" />
             </geometry>
         </collision>
@@ -257,14 +257,14 @@
             <origin xyz="0 0 0" rpy="0 0 0" />
             <geometry>
-                <mesh filename="${mesh_path}gemini336_depth_frame.STL" />
-            </geometry>
-            <material name="">
-                <color rgba="0.501960784313725 0.250980392156863 0.250980392156863 1" />
-            </material>
-        </visual>
-        <collision>
-            <origin xyz="0 0 0" rpy="0 0 0" />
-            <geometry>
-                <mesh filename="${mesh_path}gemini336_depth_frame.STL" />
+                <mesh filename="${mesh_path}camera_depth_frame.STL" />
+            </geometry>
+            <material name="">
+                <color rgba="0.501960784313725 0.250980392156863 0.250980392156863 1" />
+            </material>
+        </visual>
+        <collision>
+            <origin xyz="0 0 0" rpy="0 0 0" />
+            <geometry>
+                <mesh filename="${mesh_path}camera_depth_frame.STL" />
             </geometry>
         </collision>
@@ -286,14 +286,14 @@
             <origin xyz="0 0 0" rpy="0 0 0" />
             <geometry>
-                <mesh filename="${mesh_path}gemini336_depth_optical_frame.STL" />
-            </geometry>
-            <material name="">
-                <color rgba="0.501960784313725 0.250980392156863 0.250980392156863 1" />
-            </material>
-        </visual>
-        <collision>
-            <origin xyz="0 0 0" rpy="0 0 0" />
-            <geometry>
-                <mesh filename="${mesh_path}gemini336_depth_optical_frame.STL" />
+                <mesh filename="${mesh_path}camera_depth_optical_frame.STL" />
+            </geometry>
+            <material name="">
+                <color rgba="0.501960784313725 0.250980392156863 0.250980392156863 1" />
+            </material>
+        </visual>
+        <collision>
+            <origin xyz="0 0 0" rpy="0 0 0" />
+            <geometry>
+                <mesh filename="${mesh_path}camera_depth_optical_frame.STL" />
             </geometry>
         </collision>

File: src/bench_robot_description/urdf/gen3_macro.xacro (robot description, xacro)
@@ -487,10 +487,10 @@
       <parent link="${prefix}end_effector_link"/>
       <child link="${prefix}ee_camera_bracket_link"/>
-      <origin xyz="0 -0.009 -0.012" rpy="0 0 3.1416"/>
+      <origin xyz="0 0.0085 -0.012" rpy="0 0 0"/>
     </joint>
     <joint name="${prefix}orbbec_mount_joint" type="fixed">
       <parent link="${prefix}ee_camera_bracket_link"/>
       <child link="gemini336_link"/>
-      <origin xyz="0.025 0.045 0.015" rpy="-1.5708 -1.5708 0"/>
+      <origin xyz="0.024 0.046 0.014" rpy="-1.5708 -1.5708 0"/>
     </joint>
   </xacro:macro>
